File: FlySensei_Stack_RPi_ECAD/FlySensei_Stack_RPi_ECAD.kicad_pcb (KiCad board)
At the start: 0 parts

Commit message: PCB Design for the Raspberry PI CM4 Board (V0.1)
Parts:
- added C1: 0u1 16V, Capacitor_SMD:C_0402_1005Metric, B.Cu at (118.0, 103.2)
- added C10: 0u1 6.3V, Capacitor_SMD:C_0402_1005Metric, B.Cu at (129.0, 69.9)
- added C11: 22u 16V, Capacitor_SMD:C_0603_1608Metric, B.Cu at (99.5, 112.3)
- added C12: 1u 16V, Capacitor_SMD:C_0603_1608Metric, F.Cu at (111.3, 115.6)
- added C13: 10u 35v, Capacitor_SMD:C_0805_2012Metric, B.Cu at (152.0, 111.5)
- added C14: 10u 35v, Capacitor_SMD:C_0805_2012Metric, B.Cu at (149.8, 111.5)
- added C15: 100n 35V, Capacitor_SMD:C_0402_1005Metric, B.Cu at (136.1, 109.5)
- added C16: 10u 35V, Capacitor_SMD:C_0603_1608Metric, B.Cu at (142.4, 87.9)
- added C17: 100n 35V, Capacitor_SMD:C_0402_1005Metric, B.Cu at (146.4, 116.3)
- added C18: 100uF, Capacitor_Tantalum_SMD:CP_EIA-7343-31_Kemet-D, B.Cu at (133.1, 98.1)
- added C19: 22u 16V, Capacitor_SMD:C_0603_1608Metric, B.Cu at (137.3, 85.2)
- added C2: 0u1 16V, Capacitor_SMD:C_0402_1005Metric, B.Cu at (118.0, 104.6)
- added C20: 1nf 16V, Capacitor_SMD:C_0402_1005Metric, B.Cu at (138.4, 112.0)
- added C21: 1.2nF 16V, Capacitor_SMD:C_0402_1005Metric, B.Cu at (136.1, 110.8)
- added C22: 1nf 16V, Capacitor_SMD:C_0402_1005Metric, B.Cu at (138.4, 113.3)
- added C23: 22u 16V, Capacitor_SMD:C_0805_2012Metric, B.Cu at (145.0, 97.4)
- added C24: 22u 16V, Capacitor_SMD:C_0805_2012Metric, B.Cu at (145.0, 99.9)
- added C25: 22u 16V, Capacitor_SMD:C_0805_2012Metric, B.Cu at (145.0, 102.4)
- added C26: 22u, Capacitor_SMD:C_0805_2012Metric, F.Cu at (157.9, 72.0)
- added C27: 10u, Capacitor_SMD:C_0805_2012Metric, F.Cu at (106.0, 69.7)
- added C3: 0u1 16V, Capacitor_SMD:C_0402_1005Metric, B.Cu at (118.0, 105.9)
- added C4: 0u1 16V, Capacitor_SMD:C_0402_1005Metric, B.Cu at (118.0, 107.2)
- added C5: 0u1 6.3V, Capacitor_SMD:C_0402_1005Metric, B.Cu at (125.5, 72.1)
- added C6: 0u1 6.3V, Capacitor_SMD:C_0402_1005Metric, B.Cu at (125.5, 73.4)
- added C7: 0u1 6.3V, Capacitor_SMD:C_0402_1005Metric, B.Cu at (125.5, 74.7)
- added C8: 0u1 6.3V, Capacitor_SMD:C_0402_1005Metric, B.Cu at (125.5, 76.0)
- added C9: 0u1 6.3V, Capacitor_SMD:C_0402_1005Metric, B.Cu at (130.3, 69.9)
- added D1: LED_GRN, LED_SMD:LED_0603_1608Metric, F.Cu at (93.7, 101.6)
- added D2: LED_GRN, LED_SMD:LED_0603_1608Metric, F.Cu at (93.7, 95.2)
- added D3: LED_AMB, LED_SMD:LED_0603_1608Metric, F.Cu at (93.7, 91.0)
- added D4: LED_RED, LED_SMD:LED_0603_1608Metric, F.Cu at (93.7, 107.0)
- added D5: D_Schottky, Diode_SMD:D_SMB, F.Cu at (105.5, 114.8)
- added D6: D_Schottky, Diode_SMD:D_SMB, B.Cu at (126.2, 101.3)
- added D7: D_Schottky, Diode_SMD:D_SMB, F.Cu at (160.1, 76.8)
- added D8: LED_WHT, LED_SMD:LED_0603_1608Metric, F.Cu at (93.7, 112.0)
- added H1: MountingHole, MountingHole:MountingHole_2.7mm_M2.5_Pad_Via, F.Cu at (94.0, 126.0)
- added H2: MountingHole, MountingHole:MountingHole_2.7mm_M2.5_Pad_Via, F.Cu at (94.0, 69.0)
- added H3: MountingHole, MountingHole:MountingHole_2.7mm_M2.5_Pad_Via, F.Cu at (176.0, 69.0)
- added H4: MountingHole, MountingHole:MountingHole_2.7mm_M2.5_Pad_Via, F.Cu at (176.0, 126.0)
- added J1: Conn_01x03, Connector_PinHeader_1.00mm:PinHeader_1x03_P1.00mm_Vertical, F.Cu at (124.1, 117.9)
- added J10: Micro_SD_Card_Det, RPi_CM4IO:SDCARD_MOLEX_503398-1892, B.Cu at (108.0, 72.9)
- added J2: USB_C_Receptacle_USB2.0, Connector_USB:USB_C_Receptacle_XKB_U262-16XN-4BVC11, F.Cu at (105.5, 126.0)
- added J3: Conn_02x20_Odd_Even_Male, Connector_PinHeader_1.27mm:PinHeader_2x20_P1.27mm_Vertical_SMD, F.Cu at (105.0, 97.5)
- added J4: Conn_02x20_Odd_Even_Female, Connector_PinHeader_1.27mm:PinHeader_2x20_P1.27mm_Vertical_SMD, B.Cu at (105.0, 97.5)
- added J5: Conn_02x20_Odd_Even_Male, Connector_PinHeader_1.27mm:PinHeader_2x20_P1.27mm_Vertical_SMD, F.Cu at (165.0, 97.5)
- added J6: Conn_02x20_Odd_Even_Female, Connector_PinHeader_1.27mm:PinHeader_2x20_P1.27mm_Vertical_SMD, B.Cu at (165.0, 97.5)
- added J7: Conn_01x22_Female, Connector_FFC-FPC:Hirose_FH12-22S-0.5SH_1x22-1MP_P0.50mm_Horizontal, F.Cu at (175.0, 81.3)
- added J8: Conn_01x22_Female, Connector_FFC-FPC:Hirose_FH12-22S-0.5SH_1x22-1MP_P0.50mm_Horizontal, F.Cu at (175.0, 100.8)
- added J9: Conn_01x14_Female, Connector_FFC-FPC:Hirose_FH12-14S-0.5SH_1x14-1MP_P0.50mm_Horizontal, F.Cu at (95.0, 79.2)
- added JP1: SolderJumper_2_Open, Jumper:SolderJumper-2_P1.3mm_Open_RoundedPad1.0x1.5mm, F.Cu at (113.2, 110.8)
- added JP2: SolderJumper_2_Open, Jumper:SolderJumper-2_P1.3mm_Open_RoundedPad1.0x1.5mm, F.Cu at (122.7, 93.8)
- added JP3: SolderJumper_2_Open, Jumper:SolderJumper-2_P1.3mm_Open_RoundedPad1.0x1.5mm, F.Cu at (113.2, 105.7)
- added JP4: SolderJumper_2_Open, Jumper:SolderJumper-2_P1.3mm_Open_RoundedPad1.0x1.5mm, F.Cu at (113.2, 108.2)
- added JP5: SolderJumper_2_Open, Jumper:SolderJumper-2_P1.3mm_Open_RoundedPad1.0x1.5mm, B.Cu at (113.2, 108.2)
- added JP6: SolderJumper_2_Open, Jumper:SolderJumper-2_P1.3mm_Open_RoundedPad1.0x1.5mm, B.Cu at (99.5, 116.2)
- added JP7: SolderJumper_3_Open, Jumper:SolderJumper-3_P1.3mm_Open_RoundedPad1.0x1.5mm, B.Cu at (123.2, 79.3)
- added L1: SRN6045TA-3R3Y, Inductor_SMD:L_Bourns_SRN6045TA, B.Cu at (139.3, 103.3)
- added Q1: Q_NMOS_GSD, Package_TO_SOT_SMD:SOT-23, B.Cu at (111.7, 111.8)
- added R1: 270R, Resistor_SMD:R_0402_1005Metric, F.Cu at (93.7, 99.8)
- added R10: 62K, Resistor_SMD:R_0402_1005Metric, B.Cu at (142.4, 91.9)
- added R11: 20K 1%, Resistor_SMD:R_0402_1005Metric, B.Cu at (138.4, 110.8)
- added R12: 12K 1%, Resistor_SMD:R_0402_1005Metric, B.Cu at (136.1, 113.3)
- added R13: 2.2K 1%, Resistor_SMD:R_0402_1005Metric, B.Cu at (133.7, 113.3)
- added R14: 75K, Resistor_SMD:R_0402_1005Metric, B.Cu at (140.1, 92.7)
- added R15: 24K, Resistor_SMD:R_0402_1005Metric, B.Cu at (137.7, 92.7)
- added R16: 10K, Resistor_SMD:R_0402_1005Metric, B.Cu at (175.8, 77.3)
- added R17: 10K, Resistor_SMD:R_0402_1005Metric, B.Cu at (175.8, 76.3)
- added R18: 10K, Resistor_SMD:R_0402_1005Metric, B.Cu at (175.8, 96.8)
- added R19: 10K, Resistor_SMD:R_0402_1005Metric, B.Cu at (175.8, 95.8)
- added R2: 270R, Resistor_SMD:R_0402_1005Metric, F.Cu at (93.7, 93.4)
- added R20: 12K, Resistor_SMD:R_0402_1005Metric, F.Cu at (111.1, 73.2)
- added R21: 480, Resistor_SMD:R_0402_1005Metric, F.Cu at (93.7, 110.3)
- added R3: 270R, Resistor_SMD:R_0402_1005Metric, F.Cu at (93.7, 89.2)
- added R4: 270R, Resistor_SMD:R_0402_1005Metric, F.Cu at (93.8, 105.3)
- added R5: 4.7K, Resistor_SMD:R_0402_1005Metric, B.Cu at (97.9, 119.2)
- added R6: 900K, Resistor_SMD:R_0402_1005Metric, B.Cu at (102.6, 112.8)
- added R7: 50K, Resistor_SMD:R_0402_1005Metric, B.Cu at (102.6, 117.8)
- added R8: 10R, Resistor_SMD:R_0402_1005Metric, B.Cu at (138.4, 109.5)
- added R9: 55K, Resistor_SMD:R_0402_1005Metric, B.Cu at (142.4, 90.5)
- added SW1: SW_SPST, Button_Switch_SMD:Panasonic_EVQPUL_EVQPUC, B.Cu at (130.2, 126.4)
- added SW2: SW_SPDT, Button_Switch_SMD:SW_SPDT_PCM12, B.Cu at (93.4, 116.9)
- added SW3: SW_SPDT, Button_Switch_SMD:SW_SPDT_PCM12, B.Cu at (140.1, 126.5)
- added TP4: TestPoint, TestPoint:TestPoint_Pad_2.0x2.0mm, B.Cu at (130.4, 109.8)
- added TP6: TestPoint, TestPoint:TestPoint_Pad_2.0x2.0mm, B.Cu at (130.4, 114.0)
- added U1: ComputeModule4-CM4, RPi_CM4IO:Raspberry-Pi-4-Compute-Module, F.Cu at (118.5, 121.5)
- added U10: RT9742GGJ5, Package_TO_SOT_SMD:SOT-23-5, F.Cu at (108.1, 73.2)
- added U16: AP64501SP-13, Package_SO:SOIC-8-1EP_3.9x4.9mm_P1.27mm_EP2.95x4.9mm_Mask2.71x3.4mm_ThermalVias, B.Cu at (143.9, 111.4)
- added U2: ATtiny85V-10S, Package_SO:SOIC-8W_5.3x5.3mm_P1.27mm, B.Cu at (120.1, 111.5)
- added U3: 74LVC1G07, Package_TO_SOT_SMD:SOT-353_SC-70-5, F.Cu at (97.2, 106.2)
- added U4: G313-06329-00, AI_Coral:G313-06329-00, B.Cu at (135.0, 77.0)
- added U5: TPD2EUSB30, Package_TO_SOT_SMD:Texas_DRT-3, F.Cu at (105.5, 120.0)
- added U6: TUSB321, Package_DFN_QFN:Texas_X2QFN-12_1.6x1.6mm_P0.4mm, B.Cu at (105.2, 115.4)
- added U7: MPM3610, Package_DFN_QFN_U:MPM3610_QFN-20_5x3mm, B.Cu at (137.2, 89.3)
- added U8: TPD4EUSB30, Package_SON:USON-10_2.5x1.0mm_P0.5mm, F.Cu at (99.0, 77.4)
- added U9: TPD4EUSB30, Package_SON:USON-10_2.5x1.0mm_P0.5mm, F.Cu at (99.0, 80.9)
Routing:
- net GND: track 0.00 -> 417.4 mm, vias 0 -> 163
- net +3V3_RPI: track 0.00 -> 165.7 mm, vias 0 -> 16
- net /High Speed Interfaces/CAM_GPIO: track 0.00 -> 103.3 mm, vias 0 -> 4
- net /RPi_CM4/USB_DP: track 0.00 -> 82.4 mm, vias 0 -> 3
- net /RPi_CM4/USB_DN: track 0.00 -> 80.6 mm, vias 0 -> 3
- net /High Speed Interfaces/CAM1_SCL: track 0.00 -> 74.6 mm, vias 0 -> 3
- net /High Speed Interfaces/CAM1_SDA: track 0.00 -> 74.2 mm, vias 0 -> 3
- net /High Speed Interfaces/CAM0_SCL: track 0.00 -> 71.8 mm, vias 0 -> 4
- net /Stacking Connectors/BATT_IN: track 0.00 -> 70.6 mm, vias 0 -> 52
- net /High Speed Interfaces/CAM0_SDA: track 0.00 -> 69.7 mm, vias 0 -> 3
- net /RPi_CM4/USB_ID: track 0.00 -> 65.5 mm, vias 0 -> 1
- net /High Speed Interfaces/CAM1_MIPI.D3_P: track 0.00 -> 61.4 mm, vias 0 -> 4
- net /High Speed Interfaces/CAM1_MIPI.D3_N: track 0.00 -> 61.1 mm, vias 0 -> 4
- net /High Speed Interfaces/CAM1_MIPI.D2_P: track 0.00 -> 58.0 mm, vias 0 -> 4
- net /High Speed Interfaces/CAM1_MIPI.D2_N: track 0.00 -> 57.7 mm, vias 0 -> 4
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- added copper zone on B.Cu, net +3V3
- added copper zone on In2.Cu, net +3V3
- added copper zone on In2.Cu, net +3V3_RPI
- added copper zone on B.Cu, net +5V
- added copper zone on F.Cu, net +5V
- added copper zone on In2.Cu, net +5V
- added copper zone on B.Cu, net +BATT
- added copper zone on F.Cu, net +BATT
- added copper zone on In2.Cu, net +BATT
- added copper zone on F.Cu, net /Stacking Connectors/BATT_IN
- added copper zone on In2.Cu, net /Stacking Connectors/BATT_IN
- added copper zone on B.Cu, net GND
- added copper zone on F.Cu, net GND
- added copper zone on In1.Cu, net GND
- added copper zone on In2.Cu, net GND
- added copper zone on B.Cu, net Net-(C11-Pad1)
- added copper zone on F.Cu, net Net-(C11-Pad1)
- added copper zone on B.Cu, net Net-(C18-Pad1)
- added copper zone on B.Cu, net Net-(L1-Pad1)
- added copper zone on B.Cu, net unconnected-(U7-Pad4)
Other:
- board outline added: 90 x 65 mm
- copper layers 0 -> 4
- board text added: "1V8"
- board text added: "3V3"
- board text added: "ACT"
- board text added: "BLTH"
- board text added: "BOOT"
- board text added: "EPRM"
- board text added: "ETHERNET"
- board text added: "ON"
- board text added: "PWR"
- board text added: "USB_S"
- board text added: "WIFI"
