File: FlySensei_Stack_RPi_ECAD/FlySensei_Stack_RPi_SDCard.kicad_sch (KiCad schematic)
At the start: 4 parts, among them J10 Micro_SD_Card_Det, U10 RT9742GGJ5

Commit message: PCB Design for the Raspberry PI CM4 Board (V0.1)
Parts:
- J10: footprint CM4IO:SDCARD_MOLEX_503398-1892 -> RPi_CM4IO:SDCARD_MOLEX_503398-1892
Changed lines of the file:
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@@
     (property "Reference" "J10" (id 0) (at 144.78 57.9882 0))
     (property "Value" "Micro_SD_Card_Det" (id 1) (at 144.78 60.2996 0))
-    (property "Footprint" "CM4IO:SDCARD_MOLEX_503398-1892" (id 2) (at 198.12 60.96 0)
+    (property "Footprint" "RPi_CM4IO:SDCARD_MOLEX_503398-1892" (id 2) (at 198.12 60.96 0)
       (effects (font (size 1.27 1.27)) hide)
     )
